Commit message: added red color to common properties

File: ros2_ws/src/my_robot_description/urdf/common_properties.xacro (robot description, xacro)
@@ -1,4 +1,7 @@
 <?xml version="1.0"?>
 <robot xmlns:xacro="http://www.ros.org/wiki/xacro">
+    <material name="red">
+        <color rgba="0.5 0 0 1" />
+    </material>
     <material name="green">
         <color rgba="0 0.5 0 1" />

Commit message: most of section 6

File: ros2_ws/src/my_robot_description/urdf/common_properties.xacro (robot description, xacro)
@@ -13,3 +13,30 @@
         <color rgba="0.5 0.5 0.5 1" />
     </material>
+    <xacro:macro name="box_inertia" params="m l w h xyz rpy">
+        <inertial>
+            <origin xyz="${xyz}" rpy="${rpy}" />
+            <mass value="${m}" />
+            <inertia ixx="${(m/12) * (h*h + l*l)}" ixy="0"                        ixz="0"
+                                                   iyy="${(m/12) * (w*w + l*l)}"  iyz="0"
+                                                                                  izz="${(m/12) * (w*w + h*h)}" />
+        </inertial>
+    </xacro:macro>
+    <xacro:macro name="cylinder_inertia" params="m r h xyz rpy">
+        <inertial>
+            <origin xyz="${xyz}" rpy="${rpy}" />
+            <mass value="${m}" />
+            <inertia ixx="${(1/12) * m * (3*r*r + h*h)}"  ixy="0"                              ixz="0"
+                                                          iyy="${(1/12) * m * (3*r*r + h*h)}"  iyz="0"
+                                                                                               izz="${(1/2) * m * (r*r)}" />
+        </inertial>
+    </xacro:macro>
+    <xacro:macro name="sphere_inertia" params="m r xyz rpy">
+        <inertial>
+            <origin xyz="${xyz}" rpy="${rpy}" />
+            <mass value="${m}" />
+            <inertia ixx="${(2/5) * m * (r*r)}"  ixy="0"                     ixz="0"
+                                                 iyy="${(2/5) * m * (r*r)}"  iyz="0"
+                                                                             izz="${(2/5) * m * (r*r)}" />
+        </inertial>
+    </xacro:macro>
 </robot>

File: ros2_ws/src/my_robot_description/urdf/mobile_base.xacro (robot description, xacro)
@@ -1,14 +1,4 @@
 <?xml version="1.0"?>
 <robot xmlns:xacro="http://www.ros.org/wiki/xacro">
-    <!-- <xacro:macro name="example_macro" params="a b c">
-        <link name="dummy_link">
-            <visual>
-                <geomatry>
-                    <box size="${a} $[b} ${c}" />
-                </geomatry>
-            </visual>
-        </link>
-    </xacro:macro>
-    <xacro:example_macro a="2" b="3" c="4" /> -->
     <xacro:property name="base_length" value="0.6" />
     <xacro:property name="base_width" value="0.4" />
@@ -27,4 +17,5 @@
     </xacro:macro>
     <xacro:example_macro a="2" b="3" c="4" /> -->
+    <link name="base_footprint" />
     <link name="base_link">
         <visual>
@@ -35,4 +26,12 @@
             <material name="blue" />
         </visual>
+        <collision>
+            <geometry>
+                <box size="${base_length} ${base_width} ${base_height}" />
+            </geometry>
+            <origin xyz="0 0 ${base_height / 2.0}" rpy="0 0 0" />
+        </collision>
+        <xacro:box_inertia m="5.0" l="${2*base_length}" w="${2*base_width}" h="${2*base_height}"
+                           xyz="0 0 ${base_height / 2.0}" rpy="0 0 0" />
     </link>
     <xacro:macro name="wheel_link" params="prefix">
@@ -45,4 +44,12 @@
                 <material name="grey" />
             </visual>
+            <collision>
+                <geometry>
+                    <cylinder radius="${wheel_radius}" length="${wheel_length}" />
+                </geometry>
+                <origin xyz="0 0 0" rpy="${pi / 2.0} 0 0" />
+            </collision>
+            <xacro:cylinder_inertia m="1.0" r="${2*wheel_radius}" h="${2*wheel_length}"
+                                    xyz="0 0 0" rpy="${pi / 2.0} 0 0" />
         </link>
     </xacro:macro>
@@ -75,6 +82,12 @@
             <material name="grey" />
         </visual>
-    </link>
-    <link name="base_footprint_link">
+        <collision>
+            <geometry>
+                <sphere radius="${sphere_radius}" />
+            </geometry>
+            <origin xyz="0 0 0" rpy="0 0 0" />
+        </collision>
+        <xacro:sphere_inertia m="0.5" r="${2*sphere_radius}"
+                              xyz="0 0 0" rpy="0 0 0" />
     </link>
     <joint name="base_right_wheel_joint" type="continuous">
@@ -97,5 +110,5 @@
     </joint>
     <joint name="base_joint" type="fixed">
-        <parent link="base_footprint_link" />
+        <parent link="base_footprint" />
         <child link="base_link" />
         <origin xyz="0 0 ${wheel_radius}" rpy="0 0 0" />

File: ros2_ws/src/my_robot_description/urdf/my_robot.urdf.xacro (robot description, xacro)
@@ -3,3 +3,4 @@
     <xacro:include filename="common_properties.xacro" />
     <xacro:include filename="mobile_base.xacro" />
+    <xacro:include filename="mobile_base_gazebo.xacro" />
 </robot>
