Commit message: Done Section 6: Simulate Robot with Gazebo

File: ros2_ws/src/my_robot_description/urdf/mobile_base.xacro (robot description, xacro)
@@ -103,9 +103,8 @@
         <axis xyz="0 1 0" />
     </joint>
-    <joint name="base_caster_wheel_joint" type="continuous">
+    <joint name="base_caster_wheel_joint" type="fixed">
         <parent link="base_link" />
         <child link="caster_wheel_link" />
         <origin xyz="${base_length / 3.0} 0 -${sphere_radius}" rpy="0 0 0" />
-        <axis xyz="0 1 0" />
     </joint>
     <joint name="base_joint" type="fixed">

File: ros2_ws/src/my_robot_description/urdf/mobile_base_gazebo.xacro (robot description, xacro)
@@ -12,4 +12,6 @@
     <gazebo reference="caster_wheel_link">
         <material>Gazebo/Grey</material>
+        <mu1 value="0.1" />
+        <mu2 value="0.1" />
     </gazebo>
     <gazebo>
@@ -21,5 +23,4 @@
             <left_joint>base_left_wheel_joint</left_joint>
             <right_joint>base_right_wheel_joint</right_joint>
-            <caster_joint>base_caster_wheel_joint</caster_joint>
             <!-- kinematics -->
             <wheel_separation>0.45</wheel_separation>
