Commit message: Done Section 8: Final Project

File: ros2_ws/src/my_robot_description/urdf/camera.xacro (robot description, xacro)
@@ -24,5 +24,5 @@
         <origin xyz="${(base_length + camera_length) / 2.0} 0 ${base_height / 2.0}" rpy="0 0 0" />
     </joint>
-    <!-- #################  START example for OpenCV + rviz + gazebo ***OpevCV has different coordinates system directions*** ################# -->
+    <!--              START example for OpenCV + rviz + gazebo ***OpevCV has different coordinates system directions***              -->
     <link name="camera_link_optical">
     </link>
@@ -42,5 +42,5 @@
             ...
     -->
-    <!-- #################  END example for OpenCV + rviz + gazebo ***OpevCV has different coordinates system directions***  ################# -->
+    <!--                END example for OpenCV + rviz + gazebo ***OpevCV has different coordinates system directions***                -->
     <gazebo reference="camera_link">
         <material>Gazebo/Red</material>

File: ros2_ws/src/my_robot_description/urdf/common_properties.xacro (robot description, xacro)
@@ -1,4 +1,5 @@
 <?xml version="1.0"?>
 <robot xmlns:xacro="http://www.ros.org/wiki/xacro">
+    <!--                            Common Colors                            -->
     <material name="red">
         <color rgba="0.5 0 0 1" />
@@ -13,4 +14,11 @@
         <color rgba="0.5 0.5 0.5 1" />
     </material>
+    <material name="orange">
+        <color rgba="1 0.65 0 1" />
+    </material>
+    <material name="yellow">
+        <color rgba="1 1 0 1" />
+    </material>
+    <!--                     Common Momentun of Inertia                     -->
     <xacro:macro name="box_inertia" params="m l w h xyz rpy">
         <inertial>

File: ros2_ws/src/my_robot_description/urdf/mobile_base.xacro (robot description, xacro)
@@ -112,5 +112,4 @@
         <child link="base_link" />
         <origin xyz="0 0 ${wheel_radius}" rpy="0 0 0" />
-        <axis xyz="0 1 0" />
     </joint>
 </robot>

File: ros2_ws/src/my_robot_description/urdf/my_robot.urdf.xacro (robot description, xacro)
@@ -4,4 +4,11 @@
     <xacro:include filename="mobile_base.xacro" />
     <xacro:include filename="mobile_base_gazebo.xacro" />
+    <xacro:include filename="arm.xacro" />
+    <xacro:include filename="arm_gazebo.xacro" />
+    <joint name="mobile_base_arm_joint" type="fixed">
+        <parent link="base_link" />
+        <child link="arm_base_link" />
+        <origin xyz="${base_length / 4.0} 0 ${base_height}" rpy="0 0 0" />
+    </joint>
     <xacro:include filename="camera.xacro" />
 </robot>
